Commit message: Make it work

File: ground.urdf (robot description, URDF)
Before this commit: robot ground, 4 links, 4 joints
Joints:
- joint rot1: origin xyz=-2.5 0 1 -> xyz=0 0 0
- joint weld1: origin xyz=-2.5 0 0 -> xyz=0 0 0
- joint weld2: origin xyz=2.5 0 0 -> xyz=0 0 0

Commit message: Make ground work

File: ground.urdf (robot description, URDF)
Before this commit: robot ground, 4 links, 4 joints
Joints:
- joint rot1: origin xyz=0 0 0 -> xyz=0 0 1

Commit message: Add foot on bridge constraint

File: ground.urdf (robot description, URDF)
Before this commit: robot ground, 4 links, 4 joints
Links:
- link ground: mass 1 -> 100

Commit message: Tune solver

File: ground.urdf (robot description, URDF)
Before this commit: robot ground, 4 links, 4 joints
Links:
- link ground: mass 100 -> 1

Commit message: Add leg constraints, find solution incrementally

File: ground.urdf (robot description, URDF)
Before this commit: robot ground, 4 links, 4 joints
Links:
- link pole2: mass 1 -> 0.01

Commit message: Fix zeroing of contact force

File: ground.urdf (robot description, URDF)
Before this commit: robot ground, 4 links, 4 joints
Links:
- link ground: mass 100 -> 5
